File: design/micro-fm-radio.kicad_pcb (KiCad board)
At the start: 2 copper layers, 72.8 x 32 mm, 56 parts, among them J101 DC-IN, J102 AF-OUT, J201 ICP, Q301 MMBT3904, Q302 MMBT3904, Q303 MMBT3904, Q304 MMBT3904, SW201 B3F-1000, SW202 B3F-1000, SW203 B3F-1000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

Commit message: Fix value of C205 capacitor. Add project ID to the readme.md file.
Parts:
- C205: value 0.0001MFD -> 0.001MFD
